File: DemonEye.kicad_sch (KiCad schematic)
At the start: 51 parts, among them CN1 PicoBlade 1x06 P1.25mm, Q1 CSD25501F3, Q2 CSD25501F3, Q3 BC807-25QAZ, Q4 CSD25501F3, Q5 BC807-25QAZ, Q6 CSD25501F3, Q7 BC807-25QAZ, Q8 CSD25501F3, Q9 BC807-25QAZ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

Commit message: final revision/sync after messing up other repo and cleaning up silkscreen and pad overlap. Added EP pad for the BJT
Parts:
- Q3, Q5, Q7, Q9: symbol Transistor_BJT:Q_PNP_BEC -> PersonalSchematicSymbolLibrary:Q_PNP_BEC
Connections:
- net Gate_{B}: now also Q7.4 (C)
- net Gate_{G}: now also Q5.4 (C)
- net Gate_{R}: now also Q3.4 (C)
- net Gate_{W}: now also Q9.4 (C)
Changed lines of the file:
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@@
 	)
 	(symbol
-		(lib_id "Transistor_BJT:Q_PNP_BEC")
+		(lib_id "PersonalSchematicSymbolLibrary:Q_PNP_BEC")
 		(at 119.38 116.84 270)
 		(unit 1)
@@
 			)
 		)
-		(property "Datasheet" "https://assets.nexperia.com/documents/data-sheet/BC807-25QA_40QA.pdf"
+		(property "Datasheet" "~"
 			(at 119.38 116.84 0)
 			(effects
@@
 			)
 		)
-		(property "Description" "BJT PNP 45V 0.5A DFN1010D-3 AEC-Q100"
+		(property "Description" "PNP transistor, base/emitter/collector"
 			(at 119.38 116.84 0)
 			(effects
@@
 		(pin "1"
 		)
+		(pin "4"
+		)
 		(instances
 			(project "DemonEye"
@@
 	)
 	(symbol
-		(lib_id "Transistor_BJT:Q_PNP_BEC")
+		(lib_id "PersonalSchematicSymbolLibrary:Q_PNP_BEC")
 		(at 119.38 93.98 270)
 		(unit 1)
@@
 			)
 		)
-		(property "Datasheet" "https://assets.nexperia.com/documents/data-sheet/BC807-25QA_40QA.pdf"
+		(property "Datasheet" "~"
 			(at 119.38 93.98 0)
 			(effects
@@
 			)
 		)
-		(property "Description" "BJT PNP 45V 0.5A DFN1010D-3 AEC-Q100"
+		(property "Description" "PNP transistor, base/emitter/collector"
 			(at 119.38 93.98 0)
 			(effects
@@
 		(pin "1"
 		)
+		(pin "4"
+		)
 		(instances
 			(project "DemonEye"
@@
 	)
 	(symbol
-		(lib_id "Transistor_BJT:Q_PNP_BEC")
+		(lib_id "PersonalSchematicSymbolLibrary:Q_PNP_BEC")
 		(at 119.38 48.26 270)
 		(unit 1)
@@
 			)
 		)
-		(property "Datasheet" "https://assets.nexperia.com/documents/data-sheet/BC807-25QA_40QA.pdf"
+		(property "Datasheet" "~"
 			(at 119.38 48.26 0)
 			(effects
@@
 			)
 		)
-		(property "Description" "BJT PNP 45V 0.5A DFN1010D-3 AEC-Q100"
+		(property "Description" "PNP transistor, base/emitter/collector"
 			(at 119.38 48.26 0)
 			(effects
@@
 		(pin "1"
 		)
+		(pin "4"
+		)
 		(instances
 			(project ""
@@
 	)
 	(symbol
-		(lib_id "Transistor_BJT:Q_PNP_BEC")
+		(lib_id "PersonalSchematicSymbolLibrary:Q_PNP_BEC")
 		(at 119.38 71.12 270)
 		(unit 1)
@@
 			)
 		)
-		(property "Datasheet" "https://assets.nexperia.com/documents/data-sheet/BC807-25QA_40QA.pdf"
+		(property "Datasheet" "~"
 			(at 119.38 71.12 0)
 			(effects
@@
 			)
 		)
-		(property "Description" "BJT PNP 45V 0.5A DFN1010D-3 AEC-Q100"
+		(property "Description" "PNP transistor, base/emitter/collector"
 			(at 119.38 71.12 0)
 			(effects
@@
 		(pin "1"
 		)
+		(pin "4"
+		)
 		(instances
 			(project "DemonEye"
@@
 	)
 	(symbol
-		(lib_name "Q_PMOS_1")
 		(lib_id "PersonalSchematicSymbolLibrary:Q_PMOS")
 		(at 134.62 88.9 0)
@@
 	)
 	(symbol
-		(lib_name "QLSP06RGBXWAJ_1")
 		(lib_id "PersonalSchematicSymbolLibrary:QLSP06RGBXWAJ")
 		(at 162.56 50.8 0)
@@
 		)
 		(property "Footprint" "My Resistors:TH_0402_Nominal"
-			(at 114.3 88.9 0)
+			(at 114.3 76.2 0)
 			(effects
 				(font
 					(size 1.27 1.27)
 				)
+				(justify left bottom)
 				(hide yes)
 			)
@@
 		)
 		(property "Description" "Thermistor NTC 4.7kΩ 3500K 0402"
-			(at 114.3 88.9 0)
+			(at 114.3 81.28 0)
 			(effects
 				(font
 					(size 1.27 1.27)
 				)
+				(justify left bottom)
 				(hide yes)
 			)
 		)
 		(property "Manufacturer" "Murata Electronics"
-			(at 114.3 88.9 0)
+			(at 114.3 83.82 0)
 			(effects
 				(font
 					(size 1.27 1.27)
 				)
+				(justify left bottom)
 				(hide yes)
 			)
 		)
 		(property "Manufacturer Part Number" "NCP15XM472J03RC"
-			(at 114.3 88.9 0)
+			(at 95.25 83.82 0)
 			(effects
 				(font
 					(size 1.27 1.27)
 				)
+				(justify left bottom)
 				(hide yes)
 			)
 		)
 		(property "LCSC" "C337962"
-			(at 114.3 88.9 0)
+			(at 114.3 73.66 0)
+			(show_name yes)
 			(effects
 				(font
 					(size 1.27 1.27)
 				)
+				(justify left bottom)
 				(hide yes)
 			)
 		)
 		(property "Distributor Link 1" "https://www.digikey.com/en/products/detail/murata-electronics/NCP15XM472J03RC/588438"
-			(at 114.3 88.9 0)
+			(at 114.3 71.12 0)
 			(effects
 				(font
 					(size 1.27 1.27)
 				)
+				(justify left bottom)
 				(hide yes)
 			)
 		)
 		(property "Distributor Link 2" "https://www.mouser.com/ProductDetail/Murata-Electronics/NCP15XM472J03RC?qs=0s%252B5lLZkUHpGG9Ef%252Bzjyhg%3D%3D"
-			(at 114.3 88.9 0)
+			(at 114.3 68.58 0)
 			(effects
 				(font
 					(size 1.27 1.27)
 				)
+				(justify left bottom)
 				(hide yes)
 			)
