File: DemonEye.kicad_pcb (KiCad board)
At the start: 2 copper layers, 16 x 35.2 mm, 51 parts, among them CN1 PicoBlade 1x06 P1.25mm, Q1 CSD25501F3, Q2 CSD25501F3, Q3 BC807-25QAZ, Q4 CSD25501F3, Q5 BC807-25QAZ, Q6 CSD25501F3, Q7 BC807-25QAZ, Q8 CSD25501F3, Q9 BC807-25QAZ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

Commit message: final revision/sync after messing up other repo and cleaning up silkscreen and pad overlap. Added EP pad for the BJT
Routing:
- added copper zone on F.Cu, net /Gate_{B}
- added copper zone on F.Cu, net /Gate_{G}
- added copper zone on F.Cu, net /Gate_{R}
- added copper zone on F.Cu, net /Gate_{W}
Other:
- board text added: "v0.4.1.3"
- board text removed: "v0.4.1.2"

Commit message: Update DemonEye.kicad_pcb, DemonEye.kicad_prl, DemonEye.kicad_pro, and 8 more files
Parts:
- removed LED3: QLSP06RGBXWAJ, Personal_FootprintLibrary:QLSP06RGBXWAJ
- removed Q6, Q8: CSD25501F3, My Package_Leadless:Texas_-YJN_0.7x0.6mm_PicoStar
- removed Q7, Q9: BC807-25QAZ, My Package_Leadless:DFN1010D-3
- removed the R10 at (102.3, 66.2)
- removed R11, R14, R17: 1k0, My Resistors:R_0402_Nominal
- removed R12, R15: 5R6, My Resistors:R_0402_Nominal
- removed R13, R16: 511, My Resistors:R_0201_Dense
- removed R18, R19, R20, R21, R22, R23, R24, R25: 160, My Resistors:R_0201_Dense
- removed the R8 at (108.1, 64.5)
- removed the R9 at (103.3, 66.8)
- removed TH1, TH2, TH3, TH4: 4k7, My Resistors:TH_0402_Nominal
- added R3: 0R, My Resistors:R_0402_Nominal, F.Cu at (108.3, 71.2)
- added R4: 20Ω, My Resistors:R_0201_Dense, F.Cu at (103.3, 67.6)
- added R5: 20Ω, My Resistors:R_0201_Dense, F.Cu at (106.6, 67.6)
- added U2: TLV76701DRVx, My Package_Leadless:WSON-6-1EP_2x2mm_P0.65mm_EP1x1.6mm, F.Cu at (104.2, 71.2)
- added U3: BCR421UFDQ, DemonEye_Footprints:BCR421UFDQ, F.Cu at (102.5, 65.9)
- added U4: BCR421UFDQ, DemonEye_Footprints:BCR421UFDQ, F.Cu at (105.8, 65.9)
- added U6: BCR421UFDQ, DemonEye_Footprints:BCR421UFDQ, F.Cu at (112.7, 65.9)
- Q1, Q2, Q4: value CSD25501F3 -> PDTA123EM; footprint My Package_Leadless:Texas_-YJN_0.7x0.6mm_PicoStar -> My Package_Leadless:Diodes_DFN1006-3
- Q3: value BC807-25QAZ -> PDTA123EM; footprint My Package_Leadless:DFN1010D-3 -> My Package_Leadless:Diodes_DFN1006-3
- Q5: value BC807-25QAZ -> CSD25501F3; footprint My Package_Leadless:DFN1010D-3 -> My Package_Leadless:Texas_-YJN_0.7x0.6mm_PicoStar
- R1: renamed from R2; value 1k0 -> 1k2; footprint My Resistors:R_0402_Nominal -> My Resistors:R_0201_Dense
- R10: renamed from R1; value 1k0 -> 1k2; footprint My Resistors:R_0402_Nominal -> My Resistors:R_0201_Dense
- R2: renamed from R3; footprint My Resistors:R_0201_Nominal -> My Resistors:R_0201_Dense
- R6: value 5R6 -> 20Ω; footprint My Resistors:R_0402_Nominal -> My Resistors:R_0201_Dense
- R7: value 511 -> 20Ω
- R8: renamed from R4; value 1M43 -> 280k
- R9: renamed from R5; value 105k -> 30k9
- U5: renamed from U2; value TLV76701DRVx -> BCR421UFDQ; footprint My Package_Leadless:WSON-6-1EP_2x2mm_P0.65mm_EP1x1.6mm -> DemonEye_Footprints:BCR421UFDQ
- moved R7 11.4 mm to (113.5, 67.6), turned to 180 degrees
- moved Q4 10.1 mm to (112.2, 67.8)
- moved C3 8.37 mm to (102.0, 71.2)
- moved R8 8.27 mm to (101.0, 70.7)
- moved R9 8.27 mm to (101.0, 71.7)
- moved R6 7.17 mm to (110.2, 67.6), turned to 180 degrees
- moved Q1 7.07 mm to (102.0, 67.8)
- moved C4 6.92 mm to (106.3, 71.2), turned to -90 degrees
- moved U5 5.30 mm to (109.4, 65.9), turned to -90 degrees
- moved U1 5.05 mm to (111.2, 70.6)
- moved R2 5.03 mm to (113.6, 71.8), turned to 90 degrees
- moved R1 4.04 mm to (113.6, 70.3), turned to -90 degrees
- moved R10 3.94 mm to (102.0, 69.3), turned to -90 degrees
- moved Q2 3.89 mm to (105.2, 67.8)
- moved Q3 3.85 mm to (108.8, 67.8), turned to 180 degrees
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- renumbered C2 to C4, D6 to D1, D9 to D2, D7 to D3, D8 to D4
Connections:
- C3 pad 1: V_{OUT} -> +8V
- C4 pad 1: +12V -> +V_{BAT}
- CN1 pad 3: +12V -> +V_{BAT}
- CN1 pad 4: /D_{OUT} -> /D_{IN}
- CN1 pad 6: /D_{IN} -> /D_{OUT}
- D1 pad 1: +12V -> +V_{BAT}
- LED1 pad 1: /Red0 -> +8V_{SW}
- LED1 pad 2: /Green0 -> +8V_{SW}
- LED1 pad 3: /Blue0 -> +8V_{SW}
- LED1 pad 4: /White0 -> +8V_{SW}
- Q1 pad 1: /SRH -> /OUTR
- Q1 pad 2: V_{OUT} -> +8V_{SW}
- Q1 pad 3: /+V_{OUT_{SW}} -> /EN_{R}
- Q2 pad 1: /Gate_{R} -> /OUTG
- Q2 pad 2: /Source_{R} -> +8V_{SW}
- Q2 pad 3: /Red0 -> /EN_{G}
- Q3 pad 1: /Base_{R} -> /OUTB
- Q3 pad 2: /+V_{OUT_{SW}} -> +8V_{SW}
- Q3 pad 3: /Gate_{R} -> /EN_{B}
- Q4 pad 1: /Gate_{G} -> /OUTW
- Q4 pad 2: /Source_{G} -> +8V_{SW}
- Q4 pad 3: /Green0 -> /EN_{W}
- Q5 pad 1: /Base_{G} -> /SRH
- Q5 pad 2: /+V_{OUT_{SW}} -> +8V
- Q5 pad 3: /Gate_{G} -> +8V_{SW}
- R1 pad 2: V_{OUT} -> +8V
- R6 pad 1: /+V_{OUT_{SW}} -> GND
- R6 pad 2: /Source_{R} -> /R_{EXT_B}
- R7 pad 1: /Base_{R} -> GND
- R7 pad 2: /Source_{R} -> /R_{EXT_W}
- R8 pad 2: V_{OUT} -> +8V
- U1 pad 4: GND -> /GND0
- U5 pad 1: V_{OUT} -> unconnected-(U5-NC-Pad1)
- U5 pad 2: /FB -> /Blue2
- U5 pad 3: GND -> unconnected-(U5-NC-Pad3)
- U5 pad 4: unconnected-(U2-EN-Pad4) -> /EN_{B}
- U5 pad 5: GND -> /R_{EXT_B}
- U5 pad 6: +12V -> GND
Routing:
- net +8V_{SW}: track 0.00 -> 45.3 mm
- net +12V: track 13.5 -> 0.00 mm
- net +8V: track 0.00 -> 13.3 mm
- net /White0: track 12.9 -> 0.00 mm
- net /Blue0: track 9.46 -> 0.00 mm
- net /OUTW: track 10.3 -> 1.44 mm
- net /D_{OUT}: track 13.7 -> 5.22 mm
- net /Red2: track 1.20 -> 9.47 mm
- net /D_{IN}: track 15.0 -> 6.86 mm
- net /Green2: track 1.20 -> 8.45 mm
- net /OUTR: track 1.56 -> 8.21 mm
- net /Gate_{W}: track 6.18 -> 0.00 mm
- net /Gate_{R}: track 6.18 -> 0.00 mm
- net /Gate_{B}: track 6.18 -> 0.00 mm
- net /Gate_{G}: track 6.18 -> 0.00 mm
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- added copper zone on F.Cu, net +8V
- added copper zone on F.Cu, net +8V_{SW}
- added copper zone on F.Cu, net +V_{BAT}
- added copper zone on F.Cu, net /GND0
- added copper zone on F.Cu, net /V_{DD}
- removed copper zone on F.Cu, net +12V
- removed copper zone on F.Cu, net /+V_{OUT_{SW}}
- removed copper zone on F.Cu, net /Gate_{B}
- removed copper zone on F.Cu, net /Gate_{G}
- removed copper zone on F.Cu, net /Gate_{R}
- removed copper zone on F.Cu, net /Gate_{W}
- removed copper zone on F.Cu, net /Red3
- removed copper zone on F.Cu, net V_{OUT}
Other:
- board text added: "v0.5.0.0"
- board text removed: "v0.4.1.3"
